Commit message: Added an urdf for 4 wheel mecanum wheel robot

File: r2_description/urdf/r2.urdf (robot description, URDF)
Before this commit: robot r2, 0 links, 0 joints
Links:
- added link base_footprint
- added link base_link, mass ${base_mass}; collision box size=${base_size_x} ${base_size_y} ${base_size_z}; visual box size=${base_size_x} ${base_size_y} ${base_size_z}
- added link fl_wheel_link, mass ${wheel_mass}; collision box size=${wheel_width} ${wheel_radius*2} ${wheel_radius*2}; visual mesh filename=package://r2_description/meshes/fl_wheel_link.STL scale=0.6 0.6 0.6
- added link fr_wheel_link, mass ${wheel_mass}; collision box size=${wheel_width} ${wheel_radius*2} ${wheel_radius*2}; visual mesh filename=package://r2_description/meshes/fr_wheel_link.STL scale=0.6 0.6 0.6
- added link rl_wheel_link, mass ${wheel_mass}; collision box size=${wheel_width} ${wheel_radius*2} ${wheel_radius*2}; visual mesh filename=package://r2_description/meshes/rl_wheel_link.STL scale=0.6 0.6 0.6
- added link rr_wheel_link, mass ${wheel_mass}; collision box size=${wheel_width} ${wheel_radius*2} ${wheel_radius*2}; visual mesh filename=package://r2_description/meshes/rr_wheel_link.STL scale=0.6 0.6 0.6
Joints:
- added joint base_joint: type fixed, parent base_footprint, child base_link, origin xyz=0 0 0 rpy=0 0 0
- added joint fl_wheel_joint: type continuous, parent base_link, child fl_wheel_link, origin xyz=${-wheel_offset_x} ${-wheel_offset_y} ${wheel_offset_z} rpy=0 0 ${-M_PI/2}, axis 1 0 0
- added joint fr_wheel_joint: type continuous, parent base_link, child fr_wheel_link, origin xyz=${-wheel_offset_x} ${wheel_offset_y} ${wheel_offset_z} rpy=0 0 ${M_PI/2}, axis -1 0 0
- added joint rl_wheel_joint: type continuous, parent base_link, child rl_wheel_link, origin xyz=${wheel_offset_x} ${-wheel_offset_y} ${wheel_offset_z} rpy=0 0 ${-M_PI/2}, axis 1 0 0
- added joint rr_wheel_joint: type continuous, parent base_link, child rr_wheel_link, origin xyz=${wheel_offset_x} ${wheel_offset_y} ${wheel_offset_z} rpy=0 0 ${M_PI/2}, axis -1 0 0

Commit message: Updated the urdf and added plugins for range sensor and imu. Also implemented ros_planar move plugin.(ISSUE: angular is ignored in this plugin)

File: r2_description/urdf/r2.urdf (robot description, URDF)
Before this commit: robot r2, 6 links, 5 joints
Links:
- added link imu_link, mass 0.100; collision box size=0.02 0.02 0.02; visual box size=0.02 0.02 0.02
- added link luna_1, mass ${sensor_mass}; collision box size=${sensor_size_x} ${sensor_size_y} ${sensor_size_z}; visual box size=${sensor_size_x} ${sensor_size_y} ${sensor_size_z}
- added link luna_2, mass ${sensor_mass}; collision box size=${sensor_size_x} ${sensor_size_y} ${sensor_size_z}; visual box size=${sensor_size_x} ${sensor_size_y} ${sensor_size_z}
- added link luna_3, mass ${sensor_mass}; collision box size=${sensor_size_x} ${sensor_size_y} ${sensor_size_z}; visual box size=${sensor_size_x} ${sensor_size_y} ${sensor_size_z}
- added link luna_4, mass ${sensor_mass}; collision box size=${sensor_size_x} ${sensor_size_y} ${sensor_size_z}; visual box size=${sensor_size_x} ${sensor_size_y} ${sensor_size_z}
Joints:
- added joint imu_joint: type fixed, parent base_link, child imu_link, origin xyz=0 0 0.01 rpy=0 0 0
- added joint luna_1_joint: type fixed, parent base_link, child luna_1, origin xyz=0.22 0.1 0 rpy=0 0 0
- added joint luna_2_joint: type fixed, parent base_link, child luna_2, origin xyz=0.22 -0.1 0 rpy=0 0 0
- added joint luna_3_joint: type fixed, parent base_link, child luna_3, origin xyz=0.1 -0.2 0 rpy=0 0 ${-M_PI/2}
- added joint luna_4_joint: type fixed, parent base_link, child luna_4, origin xyz=-0.1 -0.2 0 rpy=0 0 ${-M_PI/2}
