Commit message: added holonomic drive in simulation

File: r2_description/description/body/r2_body.xacro (robot description, xacro)
@@ -28,9 +28,8 @@
             </inertial>
             </link>
-            <joint name="fl_wheel_joint" type="continuous">
+            <joint name="fl_wheel_joint" type="fixed">
                 <parent link="base_link"/>
                 <child link="fl_wheel_link"/>
                 <origin xyz="${-wheel_offset_x} ${-wheel_offset_y} ${wheel_offset_z}" rpy="0 0 ${-M_PI/2}" />
-                <axis xyz="1 0 0" rpy="0 0 0"/>
             </joint>
             <link name="fl_wheel_link">
@@ -38,25 +37,24 @@
                 <origin xyz="0 0 0" rpy="0 0 0" />
                 <geometry>
-                <mesh filename="package://r2_description/meshes/fl_wheel_link.STL" scale="0.6 0.6 0.6" />
-                </geometry>
-                <material name="darkgrey" />
-            </visual>
-            <collision>
-                <origin xyz="0 0 0" rpy="0 0 0" />
-                <geometry>
-                <box size="${wheel_width} ${wheel_radius*2} ${wheel_radius*2}" />
-                </geometry>
-            </collision>
-            <inertial>
-                <origin xyz="0 0 0" rpy="0 0 0" />
-                <mass value="${wheel_mass}" />
-                <xacro:cylinder_inertia m="${wheel_mass}" r="${wheel_radius}" w="${wheel_width}" />
-            </inertial>
-        </link>
-        <joint name="fr_wheel_joint" type="continuous">
+                <mesh filename="$(find r2_description)/meshes/fl_wheel_link.STL" scale="0.6 0.6 0.6" />
+                </geometry>
+                <material name="darkgrey" />
+            </visual>
+            <collision>
+                <origin xyz="0 0 0" rpy="0 0 0" />
+                <geometry>
+                <box size="${wheel_width} ${wheel_radius*2} ${wheel_radius*2}" />
+                </geometry>
+            </collision>
+            <inertial>
+                <origin xyz="0 0 0" rpy="0 0 0" />
+                <mass value="${wheel_mass}" />
+                <xacro:cylinder_inertia m="${wheel_mass}" r="${wheel_radius}" w="${wheel_width}" />
+            </inertial>
+        </link>
+        <joint name="fr_wheel_joint" type="fixed">
             <parent link="base_link"/>
             <child link="fr_wheel_link"/>
             <origin xyz="${-wheel_offset_x} ${wheel_offset_y} ${wheel_offset_z}" rpy="0 0 ${M_PI/2}" />
-            <axis xyz="-1 0 0" rpy="0 0 0"/>
         </joint>
         <link name="fr_wheel_link">
@@ -64,25 +62,24 @@
                 <origin xyz="0 0 0" rpy="0 0 0" />
                 <geometry>
-                <mesh filename="package://r2_description/meshes/fr_wheel_link.STL" scale="0.6 0.6 0.6" />
-                </geometry>
-                <material name="darkgrey" />
-            </visual>
-            <collision>
-                <origin xyz="0 0 0" rpy="0 0 0" />
-                <geometry>
-                <box size="${wheel_width} ${wheel_radius*2} ${wheel_radius*2}" />
-                </geometry>
-            </collision>
-            <inertial>
-                <origin xyz="0 0 0" rpy="0 0 0" />
-                <mass value="${wheel_mass}" />
-                <xacro:cylinder_inertia m="${wheel_mass}" r="${wheel_radius}" w="${wheel_width}" />
-            </inertial>
-            </link>
-            <joint name="rl_wheel_joint" type="continuous">
+                <mesh filename="$(find r2_description)/meshes/fr_wheel_link.STL" scale="0.6 0.6 0.6" />
+                </geometry>
+                <material name="darkgrey" />
+            </visual>
+            <collision>
+                <origin xyz="0 0 0" rpy="0 0 0" />
+                <geometry>
+                <box size="${wheel_width} ${wheel_radius*2} ${wheel_radius*2}" />
+                </geometry>
+            </collision>
+            <inertial>
+                <origin xyz="0 0 0" rpy="0 0 0" />
+                <mass value="${wheel_mass}" />
+                <xacro:cylinder_inertia m="${wheel_mass}" r="${wheel_radius}" w="${wheel_width}" />
+            </inertial>
+            </link>
+            <joint name="rl_wheel_joint" type="fixed">
                 <parent link="base_link"/>
                 <child link="rl_wheel_link"/>
                 <origin xyz="${wheel_offset_x} ${-wheel_offset_y} ${wheel_offset_z}" rpy="0 0 ${-M_PI/2}" />
-                <axis xyz="1 0 0" rpy="0 0 0"/>
             </joint>
             <link name="rl_wheel_link">
@@ -90,25 +87,24 @@
                 <origin xyz="0 0 0" rpy="0 0 0" />
                 <geometry>
-                <mesh filename="package://r2_description/meshes/rl_wheel_link.STL" scale="0.6 0.6 0.6" />
-                </geometry>
-                <material name="darkgrey" />
-            </visual>
-            <collision>
-                <origin xyz="0 0 0" rpy="0 0 0" />
-                <geometry>
-                <box size="${wheel_width} ${wheel_radius*2} ${wheel_radius*2}" />
-                </geometry>
-            </collision>
-            <inertial>
-                <origin xyz="0 0 0" rpy="0 0 0" />
-                <mass value="${wheel_mass}" />
-                <xacro:cylinder_inertia m="${wheel_mass}" r="${wheel_radius}" w="${wheel_width}" />
-            </inertial>
-            </link>
-            <joint name="rr_wheel_joint" type="continuous">
+                <mesh filename="$(find r2_description)/meshes/rl_wheel_link.STL" scale="0.6 0.6 0.6" />
+                </geometry>
+                <material name="darkgrey" />
+            </visual>
+            <collision>
+                <origin xyz="0 0 0" rpy="0 0 0" />
+                <geometry>
+                <box size="${wheel_width} ${wheel_radius*2} ${wheel_radius*2}" />
+                </geometry>
+            </collision>
+            <inertial>
+                <origin xyz="0 0 0" rpy="0 0 0" />
+                <mass value="${wheel_mass}" />
+                <xacro:cylinder_inertia m="${wheel_mass}" r="${wheel_radius}" w="${wheel_width}" />
+            </inertial>
+            </link>
+            <joint name="rr_wheel_joint" type="fixed">
                 <parent link="base_link"/>
                 <child link="rr_wheel_link"/>
                 <origin xyz="${wheel_offset_x} ${wheel_offset_y} ${wheel_offset_z}" rpy="0 0 ${M_PI/2}" />
-                <axis xyz="-1 0 0" rpy="0 0 0"/>
             </joint>
             <link name="rr_wheel_link">
@@ -116,5 +112,5 @@
                 <origin xyz="0 0 0" rpy="0 0 0" />
                 <geometry>
-                <mesh filename="package://r2_description/meshes/rr_wheel_link.STL" scale="0.6 0.6 0.6" />
+                <mesh filename="$(find r2_description)/meshes/rr_wheel_link.STL" scale="0.6 0.6 0.6" />
                 </geometry>
                 <material name="darkgrey" />

Commit message: added sensors

File: r2_description/description/body/r2_body.xacro (robot description, xacro)
@@ -228,4 +228,30 @@
             </inertial>
         </link>
+        <!-- IMU LINK AT CENTER OF ROBOT -->
+    <joint name="imu_joint" type="fixed">
+        <parent link="base_link" />
+        <child link="imu_link" />
+        <origin xyz="0 0 0.01" rpy="0 0 0" />
+    </joint>
+  <link name="imu_link">
+    <visual>
+      <origin xyz="0 0 0" rpy="0 0 0" />
+      <geometry>
+        <box size="0.02 0.02 0.02" />
+      </geometry>
+      <material name="grey" />
+    </visual>
+    <collision>
+      <origin xyz="0 0 0" rpy="0 0 0" />
+      <geometry>
+        <box size="0.02 0.02 0.02" />
+      </geometry>
+    </collision>
+    <inertial>
+      <origin xyz="0.0 0.0 0.0" rpy="0.0 0.0 0.0"/>
+      <mass value="0.100"/>
+      <xacro:box_inertia m="0.100" x="0.02" y="0.02" z="0.02"/>
+    </inertial>
+  </link>
     </xacro:macro>
 </robot>

File: r2_description/description/gazebo.xacro (robot description, xacro)
@@ -12,3 +12,234 @@
         </plugin>
   </gazebo>
+  <gazebo reference="luna_1">
+    <sensor name="luna_1" type="ray">
+        <always_on>true</always_on>
+        <visualize>true</visualize>
+        <pose>0.0 0 0.0 0 0 0</pose>
+        <update_rate>5</update_rate>
+        <ray>
+            <scan>
+                <horizontal>
+                    <samples>5</samples>
+                    <resolution>1.0</resolution>
+                    <min_angle>0</min_angle>
+                    <max_angle>0</max_angle>
+                </horizontal>
+                <vertical>
+                    <samples>5</samples>
+                    <resolution>1.0</resolution>
+                    <min_angle>0.0</min_angle>
+                    <max_angle>0.0</max_angle>
+                </vertical>
+            </scan>
+            <range>
+                <min>0.02</min>
+                <max>8</max>
+                <resolution>0.01</resolution>
+            </range>
+            <noise>
+                <type>gaussian</type>
+                <mean>0.0</mean>
+                <stddev>0.01</stddev>
+            </noise>
+        </ray>
+        <plugin name="luna_1" filename="libgazebo_ros_ray_sensor.so">
+            <ros>
+                <namespace>distance</namespace>
+                <remapping>~/out:=luna_1</remapping>
+            </ros>
+            <output_type>sensor_msgs/Range</output_type>
+            <radiation_type>ultrasound</radiation_type>
+            <frame_name>luna_1_dist_sensor</frame_name>
+        </plugin>
+    </sensor>
+    <material>Gazebo/Blue</material>
+</gazebo>
+<gazebo reference="luna_2">
+    <sensor name="luna_2" type="ray">
+        <always_on>true</always_on>
+        <visualize>true</visualize>
+        <pose>0.0 0 0.0 0 0 0</pose>
+        <update_rate>5</update_rate>
+        <ray>
+            <scan>
+                <horizontal>
+                    <samples>5</samples>
+                    <resolution>1.0</resolution>
+                    <min_angle>0</min_angle>
+                    <max_angle>0</max_angle>
+                </horizontal>
+                <vertical>
+                    <samples>5</samples>
+                    <resolution>1.0</resolution>
+                    <min_angle>0.0</min_angle>
+                    <max_angle>0.0</max_angle>
+                </vertical>
+            </scan>
+            <range>
+                <min>0.02</min>
+                <max>8</max>
+                <resolution>0.01</resolution>
+            </range>
+            <noise>
+                <type>gaussian</type>
+                <mean>0.0</mean>
+                <stddev>0.01</stddev>
+            </noise>
+        </ray>
+        <plugin name="luna_2" filename="libgazebo_ros_ray_sensor.so">
+            <ros>
+                <namespace>distance</namespace>
+                <remapping>~/out:=luna_2</remapping>
+            </ros>
+            <output_type>sensor_msgs/Range</output_type>
+            <radiation_type>ultrasound</radiation_type>
+            <frame_name>luna_2_dist_sensor</frame_name>
+        </plugin>
+    </sensor>
+    <material>Gazebo/Blue</material>
+</gazebo>
+<gazebo reference="luna_3">
+    <sensor name="luna_3" type="ray">
+        <always_on>true</always_on>
+        <visualize>true</visualize>
+        <pose>0.0 0 0.0 0 0 0</pose>
+        <update_rate>5</update_rate>
+        <ray>
+            <scan>
+                <horizontal>
+                    <samples>5</samples>
+                    <resolution>1.0</resolution>
+                    <min_angle>0</min_angle>
+                    <max_angle>0</max_angle>
+                </horizontal>
+                <vertical>
+                    <samples>5</samples>
+                    <resolution>1.0</resolution>
+                    <min_angle>0.0</min_angle>
+                    <max_angle>0.0</max_angle>
+                </vertical>
+            </scan>
+            <range>
+                <min>0.02</min>
+                <max>8</max>
+                <resolution>0.01</resolution>
+            </range>
+            <noise>
+                <type>gaussian</type>
+                <mean>0.0</mean>
+                <stddev>0.01</stddev>
+            </noise>
+        </ray>
+        <plugin name="luna_3" filename="libgazebo_ros_ray_sensor.so">
+            <ros>
+                <namespace>distance</namespace>
+                <remapping>~/out:=luna_3</remapping>
+            </ros>
+            <output_type>sensor_msgs/Range</output_type>
+            <radiation_type>ultrasound</radiation_type>
+            <frame_name>luna_3_dist_sensor</frame_name>
+        </plugin>
+    </sensor>
+    <material>Gazebo/Blue</material>
+</gazebo>
+<gazebo reference="luna_4">
+    <sensor name="luna_4" type="ray">
+        <always_on>true</always_on>
+        <visualize>true</visualize>
+        <pose>0.0 0 0.0 0 0 0</pose>
+        <update_rate>5</update_rate>
+        <ray>
+            <scan>
+                <horizontal>
+                    <samples>5</samples>
+                    <resolution>1.0</resolution>
+                    <min_angle>0</min_angle>
+                    <max_angle>0</max_angle>
+                </horizontal>
+                <vertical>
+                    <samples>5</samples>
+                    <resolution>1.0</resolution>
+                    <min_angle>0.0</min_angle>
+                    <max_angle>0.0</max_angle>
+                </vertical>
+            </scan>
+            <range>
+                <min>0.02</min>
+                <max>8</max>
+                <resolution>0.01</resolution>
+            </range>
+            <noise>
+                <type>gaussian</type>
+                <mean>0.0</mean>
+                <stddev>0.01</stddev>
+            </noise>
+        </ray>
+        <plugin name="luna_4" filename="libgazebo_ros_ray_sensor.so">
+            <ros>
+                <namespace>distance</namespace>
+                <remapping>~/out:=luna_4</remapping>
+            </ros>
+            <output_type>sensor_msgs/Range</output_type>
+            <radiation_type>ultrasound</radiation_type>
+            <frame_name>luna_4_dist_sensor</frame_name>
+        </plugin>
+    </sensor>
+    <material>Gazebo/Blue</material>
+</gazebo>
+<gazebo reference="imu_link">
+    <sensor name="r2_imu" type="imu">
+        <always_on>true</always_on>
+        <update_rate>100</update_rate>
+        <imu>
+          <angular_velocity>
+            <x>
+              <noise type="gaussian">
+                <mean>0.0</mean>
+                <stddev>2e-4</stddev>
+              </noise>
+            </x>
+            <y>
+              <noise type="gaussian">
+                <mean>0.0</mean>
+                <stddev>2e-4</stddev>
+              </noise>
+            </y>
+            <z>
+              <noise type="gaussian">
+                <mean>0.0</mean>
+                <stddev>2e-4</stddev>
+              </noise>
+            </z>
+          </angular_velocity>
+          <linear_acceleration>
+            <x>
+              <noise type="gaussian">
+                <mean>0.0</mean>
+                <stddev>1.7e-2</stddev>
+              </noise>
+            </x>
+            <y>
+              <noise type="gaussian">
+                <mean>0.0</mean>
+                <stddev>1.7e-2</stddev>
+              </noise>
+            </y>
+            <z>
+              <noise type="gaussian">
+                <mean>0.0</mean>
+                <stddev>1.7e-2</stddev>
+              </noise>
+            </z>
+          </linear_acceleration>
+        </imu>
+        <plugin name="imu_plugin" filename="libgazebo_ros_imu_sensor.so">
+            <ros>
+                <namespace>imu</namespace>
+                <remapping>~/out:=data</remapping>
+            </ros>
+            <initial_orientation_as_reference>true</initial_orientation_as_reference>
+        </plugin>
+    </sensor>
+</gazebo>
 </robot>
