Commit message: Added robocon arena,r2
+blue balls,purple balls

File: r2_description/description/body/flat_bot.xacro (robot description, xacro)
@@ -234,23 +234,23 @@
         <origin xyz="0 0 0.01" rpy="0 0 0" />
     </joint>
-  <link name="imu_link">
-    <visual>
-      <origin xyz="0 0 0" rpy="0 0 0" />
-      <geometry>
-        <box size="0.02 0.02 0.02" />
-      </geometry>
-      <material name="grey" />
-    </visual>
-    <collision>
-      <origin xyz="0 0 0" rpy="0 0 0" />
-      <geometry>
-        <box size="0.02 0.02 0.02" />
-      </geometry>
-    </collision>
-    <inertial>
-      <origin xyz="0.0 0.0 0.0" rpy="0.0 0.0 0.0"/>
-      <mass value="0.100"/>
-      <xacro:box_inertia m="0.100" x="0.02" y="0.02" z="0.02"/>
-    </inertial>
+    <link name="imu_link">
+        <visual>
+            <origin xyz="0 0 0" rpy="0 0 0" />
+            <geometry>
+                <box size="0.02 0.02 0.02" />
+            </geometry>
+            <material name="grey" />
+        </visual>
+        <collision>
+            <origin xyz="0 0 0" rpy="0 0 0" />
+            <geometry>
+                <box size="0.02 0.02 0.02" />
+            </geometry>
+        </collision>
+        <inertial>
+        <origin xyz="0.0 0.0 0.0" rpy="0.0 0.0 0.0"/>
+        <mass value="0.100"/>
+        <xacro:box_inertia m="0.100" x="0.02" y="0.02" z="0.02"/>
+        </inertial>
   </link>
     </xacro:macro>

File: r2_description/description/body/r2.xacro (robot description, xacro)
@@ -33,5 +33,5 @@
                 <mesh filename="file://$(find r2_description)/meshes/wheel_fl_1.stl" scale="0.001 0.001 0.001"/>
               </geometry>
-              <material name="silver"/>
+              <material name="black"/>
             </visual>
             <collision>
@@ -53,5 +53,5 @@
                 <mesh filename="file://$(find r2_description)/meshes/wheel_bl_1.stl" scale="0.001 0.001 0.001"/>
               </geometry>
-              <material name="silver"/>
+              <material name="black"/>
             </visual>
             <collision>
@@ -73,5 +73,5 @@
                 <mesh filename="file://$(find r2_description)/meshes/wheel_fr_1.stl" scale="0.001 0.001 0.001"/>
               </geometry>
-              <material name="silver"/>
+              <material name="black"/>
             </visual>
             <collision>
@@ -93,5 +93,5 @@
                 <mesh filename="file://$(find r2_description)/meshes/wheel_br_1.stl" scale="0.001 0.001 0.001"/>
               </geometry>
-              <material name="silver"/>
+              <material name="black"/>
             </visual>
             <collision>

File: r2_description/description/common.xacro (robot description, xacro)
@@ -10,7 +10,53 @@
     <color rgba="0.0 0.0 0.8 1.0" />
 </material>
+<!-- <xacro:property name="body_color" value="Gazebo/Silver" /> -->
 <material name="silver">
     <color rgba="0.700 0.700 0.700 1.000"/>
   </material>
+  <material name="black">
+    <color rgba="0 0 0 1"/>
+  </material>
+  <gazebo reference="base_link">
+    <material>Gazebo/Grey</material>
+  </gazebo>
+  <gazebo reference="wheel_fl_1">
+    <material>Gazebo/Black</material>
+  </gazebo>
+  <gazebo reference="wheel_bl_1">
+    <material>Gazebo/Black</material>
+  </gazebo>
+  <gazebo reference="wheel_fr_1">
+    <material>Gazebo/Black</material>
+  </gazebo>
+  <gazebo reference="wheel_br_1">
+    <material>Gazebo/Black</material>
+  </gazebo>
+  <gazebo reference="lidar_lf_1">
+    <material>Gazebo/Silver</material>
+  </gazebo>
+  <gazebo reference="lidar_lb_1">
+    <material>Gazebo/Silver</material>
+  </gazebo>
+  <gazebo reference="lidar_fl_1">
+    <material>Gazebo/Silver</material>
+  </gazebo>
+  <gazebo reference="lidar_fr_1">
+    <material>Gazebo/Silver</material>
+  </gazebo>
+  <gazebo reference="lidar_rf_1">
+    <material>Gazebo/Silver</material>
+  </gazebo>
+  <gazebo reference="lidar_rb_1">
+    <material>Gazebo/Silver</material>
+  </gazebo>
+  <gazebo reference="lift_1">
+    <material>Gazebo/Turquoise</material>
+  </gazebo>
+  <gazebo reference="claw_left_1">
+    <material>Gazebo/Turquoise</material>
+  </gazebo>
+  <gazebo reference="claw_right_1">
+    <material>Gazebo/Turquoise</material>
+  </gazebo>
 <xacro:property name="M_PI" value="3.1415926535897931" />
 <xacro:property name="M_PI_2" value="1.570796327" />
