Commit message: added luna, imu sensor to r2

File: r2_description/description/body/r2.xacro (robot description, xacro)
@@ -2,4 +2,10 @@
 <robot xmlns:xacro="http://www.ros.org/wiki/xacro" name="r2">
     <xacro:macro name="r2" >
+      <link name="base_footprint"/>
+      <joint name="base_joint" type="fixed">
+        <parent link="base_footprint" />
+        <child link="base_link" />
+        <origin xyz="0 0 0.126" rpy="0 0 0" />
+      </joint>
         <link name="base_link">
             <inertial>
@@ -109,5 +115,5 @@
             </inertial>
             <visual>
-              <origin xyz="-0.052465 -0.19 0.0745" rpy="0 0 0"/>
+              <origin xyz="-0.052465 -0.19 0.0745" rpy="0 0 ${pi/2}"/>
               <geometry>
                 <mesh filename="file://$(find r2_description)/meshes/lidar_lf_1.stl" scale="0.001 0.001 0.001"/>
@@ -116,5 +122,5 @@
             </visual>
             <collision>
-              <origin xyz="-0.052465 -0.19 0.0745" rpy="0 0 0"/>
+              <origin xyz="-0.052465 -0.19 0.0745" rpy="0 0 ${pi/2}"/>
               <geometry>
                 <mesh filename="file://$(find r2_description)/meshes/lidar_lf_1.stl" scale="0.001 0.001 0.001"/>
@@ -129,5 +135,5 @@
             </inertial>
             <visual>
-              <origin xyz="0.047535 -0.19 0.0745" rpy="0 0 0"/>
+              <origin xyz="0.047535 -0.19 0.0745" rpy="0 0 ${pi/2}"/>
               <geometry>
                 <mesh filename="file://$(find r2_description)/meshes/lidar_lb_1.stl" scale="0.001 0.001 0.001"/>
@@ -136,5 +142,5 @@
             </visual>
             <collision>
-              <origin xyz="0.047535 -0.19 0.0745" rpy="0 0 0"/>
+              <origin xyz="0.047535 -0.19 0.0745" rpy="0 0 ${pi/2}"/>
               <geometry>
                 <mesh filename="file://$(find r2_description)/meshes/lidar_lb_1.stl" scale="0.001 0.001 0.001"/>
@@ -189,5 +195,5 @@
             </inertial>
             <visual>
-              <origin xyz="-0.052465 0.19 0.0745" rpy="0 0 0"/>
+              <origin xyz="-0.052465 0.19 0.0745" rpy="0 0 -${pi/2}"/>
               <geometry>
                 <mesh filename="file://$(find r2_description)/meshes/lidar_rf_1.stl" scale="0.001 0.001 0.001"/>
@@ -196,5 +202,5 @@
             </visual>
             <collision>
-              <origin xyz="-0.052465 0.19 0.0745" rpy="0 0 0"/>
+              <origin xyz="-0.052465 0.19 0.0745" rpy="0 0 -${pi/2}"/>
               <geometry>
                 <mesh filename="file://$(find r2_description)/meshes/lidar_rf_1.stl" scale="0.001 0.001 0.001"/>
@@ -209,5 +215,5 @@
             </inertial>
             <visual>
-              <origin xyz="0.047535 0.19 0.0745" rpy="0 0 0"/>
+              <origin xyz="0.047535 0.19 0.0745" rpy="0 0 -${pi/2}"/>
               <geometry>
                 <mesh filename="file://$(find r2_description)/meshes/lidar_rb_1.stl" scale="0.001 0.001 0.001"/>
@@ -216,5 +222,5 @@
             </visual>
             <collision>
-              <origin xyz="0.047535 0.19 0.0745" rpy="0 0 0"/>
+              <origin xyz="0.047535 0.19 0.0745" rpy="0 0 -${pi/2}"/>
               <geometry>
                 <mesh filename="file://$(find r2_description)/meshes/lidar_rb_1.stl" scale="0.001 0.001 0.001"/>
@@ -307,10 +313,10 @@
           </joint>
           <joint name="lidar_lf" type="fixed">
-            <origin xyz="0.052465 0.19 -0.0745" rpy="0 0 0"/>
+            <origin xyz="0.052465 0.19 -0.0745" rpy="0 0 ${pi/2}"/>
             <parent link="base_link"/>
             <child link="lidar_lf_1"/>
           </joint>
           <joint name="lidar_lb" type="fixed">
-            <origin xyz="-0.047535 0.19 -0.0745" rpy="0 0 0"/>
+            <origin xyz="-0.047535 0.19 -0.0745" rpy="0 0 ${pi/2}"/>
             <parent link="base_link"/>
             <child link="lidar_lb_1"/>
@@ -327,10 +333,10 @@
           </joint>
           <joint name="lidar_rf" type="fixed">
-            <origin xyz="0.052465 -0.19 -0.0745" rpy="0 0 0"/>
+            <origin xyz="0.052465 -0.19 -0.0745" rpy="0 0 -${pi/2}"/>
             <parent link="base_link"/>
             <child link="lidar_rf_1"/>
           </joint>
           <joint name="lidar_rb" type="fixed">
-            <origin xyz="-0.047535 -0.19 -0.0745" rpy="0 0 0"/>
+            <origin xyz="-0.047535 -0.19 -0.0745" rpy="0 0 -${pi/2}"/>
             <parent link="base_link"/>
             <child link="lidar_rb_1"/>
@@ -355,4 +361,23 @@
             <axis xyz="0.0 0.0 1.0"/>
           </joint>
+        <joint name="camera_joint" type="fixed">
+            <parent link="base_link" />
+            <child link="camera_link"/>
+            <origin xyz="0.305 0 0.08" rpy="0 0 0"/>
+        </joint>
+        <link name="camera_link">
+             <visual>
+                <geometry>
+                    <box size="0.010 0.03 0.03"/>
+                </geometry>
+                <material name="red"/>
+            </visual>
+        </link>
+        <joint name="camera_optical_joint" type="fixed">
+            <parent link="camera_link" />
+            <child link="camera_link_optical"/>
+            <origin xyz="0 0 0" rpy="${-pi/2} 0 ${-pi/2}"/>
+        </joint>
+        <link name="camera_link_optical"></link>
     </xacro:macro>
 </robot>

File: r2_description/description/flat_bot.urdf.xacro (robot description, xacro)
@@ -5,3 +5,7 @@
     <xacro:flat_bot/>
     <xacro:include filename="gazebo.xacro"/>
+    <xacro:luna prefix="luna_1"/>
+    <xacro:luna prefix="luna_2"/>
+    <xacro:luna prefix="luna_3"/>
+    <xacro:luna prefix="luna_4"/>
 </robot>

File: r2_description/description/gazebo.xacro (robot description, xacro)
@@ -12,180 +12,50 @@
         </plugin>
   </gazebo>
-  <gazebo reference="luna_1">
-    <sensor name="luna_1" type="ray">
-        <always_on>true</always_on>
-        <visualize>true</visualize>
-        <pose>0.0 0 0.0 0 0 0</pose>
-        <update_rate>5</update_rate>
-        <ray>
-            <scan>
-                <horizontal>
-                    <samples>5</samples>
-                    <resolution>1.0</resolution>
-                    <min_angle>0</min_angle>
-                    <max_angle>0</max_angle>
-                </horizontal>
-                <vertical>
-                    <samples>5</samples>
-                    <resolution>1.0</resolution>
-                    <min_angle>0.0</min_angle>
-                    <max_angle>0.0</max_angle>
-                </vertical>
-            </scan>
-            <range>
-                <min>0.02</min>
-                <max>8</max>
-                <resolution>0.01</resolution>
-            </range>
-            <noise>
-                <type>gaussian</type>
-                <mean>0.0</mean>
-                <stddev>0.01</stddev>
-            </noise>
-        </ray>
-        <plugin name="luna_1" filename="libgazebo_ros_ray_sensor.so">
-            <ros>
-                <namespace>distance</namespace>
-                <remapping>~/out:=luna_1</remapping>
-            </ros>
-            <output_type>sensor_msgs/Range</output_type>
-            <radiation_type>ultrasound</radiation_type>
-            <frame_name>luna_1_dist_sensor</frame_name>
-        </plugin>
-    </sensor>
-    <material>Gazebo/Blue</material>
-</gazebo>
-<gazebo reference="luna_2">
-    <sensor name="luna_2" type="ray">
-        <always_on>true</always_on>
-        <visualize>true</visualize>
-        <pose>0.0 0 0.0 0 0 0</pose>
-        <update_rate>5</update_rate>
-        <ray>
-            <scan>
-                <horizontal>
-                    <samples>5</samples>
-                    <resolution>1.0</resolution>
-                    <min_angle>0</min_angle>
-                    <max_angle>0</max_angle>
-                </horizontal>
-                <vertical>
-                    <samples>5</samples>
-                    <resolution>1.0</resolution>
-                    <min_angle>0.0</min_angle>
-                    <max_angle>0.0</max_angle>
-                </vertical>
-            </scan>
-            <range>
-                <min>0.02</min>
-                <max>8</max>
-                <resolution>0.01</resolution>
-            </range>
-            <noise>
-                <type>gaussian</type>
-                <mean>0.0</mean>
-                <stddev>0.01</stddev>
-            </noise>
-        </ray>
-        <plugin name="luna_2" filename="libgazebo_ros_ray_sensor.so">
-            <ros>
-                <namespace>distance</namespace>
-                <remapping>~/out:=luna_2</remapping>
-            </ros>
-            <output_type>sensor_msgs/Range</output_type>
-            <radiation_type>ultrasound</radiation_type>
-            <frame_name>luna_2_dist_sensor</frame_name>
-        </plugin>
-    </sensor>
-    <material>Gazebo/Blue</material>
-</gazebo>
-<gazebo reference="luna_3">
-    <sensor name="luna_3" type="ray">
-        <always_on>true</always_on>
-        <visualize>true</visualize>
-        <pose>0.0 0 0.0 0 0 0</pose>
-        <update_rate>5</update_rate>
-        <ray>
-            <scan>
-                <horizontal>
-                    <samples>5</samples>
-                    <resolution>1.0</resolution>
-                    <min_angle>0</min_angle>
-                    <max_angle>0</max_angle>
-                </horizontal>
-                <vertical>
-                    <samples>5</samples>
-                    <resolution>1.0</resolution>
-                    <min_angle>0.0</min_angle>
-                    <max_angle>0.0</max_angle>
-                </vertical>
-            </scan>
-            <range>
-                <min>0.02</min>
-                <max>8</max>
-                <resolution>0.01</resolution>
-            </range>
-            <noise>
-                <type>gaussian</type>
-                <mean>0.0</mean>
-                <stddev>0.01</stddev>
-            </noise>
-        </ray>
-        <plugin name="luna_3" filename="libgazebo_ros_ray_sensor.so">
-            <ros>
-                <namespace>distance</namespace>
-                <remapping>~/out:=luna_3</remapping>
-            </ros>
-            <output_type>sensor_msgs/Range</output_type>
-            <radiation_type>ultrasound</radiation_type>
-            <frame_name>luna_3_dist_sensor</frame_name>
-        </plugin>
-    </sensor>
-    <material>Gazebo/Blue</material>
-</gazebo>
-<gazebo reference="luna_4">
-    <sensor name="luna_4" type="ray">
-        <always_on>true</always_on>
-        <visualize>true</visualize>
-        <pose>0.0 0 0.0 0 0 0</pose>
-        <update_rate>5</update_rate>
-        <ray>
-            <scan>
-                <horizontal>
-                    <samples>5</samples>
-                    <resolution>1.0</resolution>
-                    <min_angle>0</min_angle>
-                    <max_angle>0</max_angle>
-                </horizontal>
-                <vertical>
-                    <samples>5</samples>
-                    <resolution>1.0</resolution>
-                    <min_angle>0.0</min_angle>
-                    <max_angle>0.0</max_angle>
-                </vertical>
-            </scan>
-            <range>
-                <min>0.02</min>
-                <max>8</max>
-                <resolution>0.01</resolution>
-            </range>
-            <noise>
-                <type>gaussian</type>
-                <mean>0.0</mean>
-                <stddev>0.01</stddev>
-            </noise>
-        </ray>
-        <plugin name="luna_4" filename="libgazebo_ros_ray_sensor.so">
-            <ros>
-                <namespace>distance</namespace>
-                <remapping>~/out:=luna_4</remapping>
-            </ros>
-            <output_type>sensor_msgs/Range</output_type>
-            <radiation_type>ultrasound</radiation_type>
-            <frame_name>luna_4_dist_sensor</frame_name>
-        </plugin>
-    </sensor>
-    <material>Gazebo/Blue</material>
-</gazebo>
+  <xacro:macro name="luna" params="prefix">
+    <gazebo reference="${prefix}">
+        <sensor name="${prefix}" type="ray">
+            <always_on>true</always_on>
+            <visualize>true</visualize>
+            <pose>0.0 0 0.0 0 0 0</pose>
+            <update_rate>5</update_rate>
+            <ray>
+                <scan>
+                    <horizontal>
+                        <samples>5</samples>
+                        <resolution>1.0</resolution>
+                        <min_angle>0</min_angle>
+                        <max_angle>0</max_angle>
+                    </horizontal>
+                    <vertical>
+                        <samples>5</samples>
+                        <resolution>1.0</resolution>
+                        <min_angle>0.0</min_angle>
+                        <max_angle>0.0</max_angle>
+                    </vertical>
+                </scan>
+                <range>
+                    <min>0.02</min>
+                    <max>8</max>
+                    <resolution>0.01</resolution>
+                </range>
+                <noise>
+                    <type>gaussian</type>
+                    <mean>0.0</mean>
+                    <stddev>0.01</stddev>
+                </noise>
+            </ray>
+            <plugin name="${prefix}" filename="libgazebo_ros_ray_sensor.so">
+                <ros>
+                    <namespace>distance</namespace>
+                    <remapping>~/out:=${prefix}</remapping>
+                </ros>
+                <output_type>sensor_msgs/Range</output_type>
+                <radiation_type>ultrasound</radiation_type>
+                <frame_name>${prefix}_dist_sensor</frame_name>
+            </plugin>
+        </sensor>
+        <material>Gazebo/Blue</material>
+    </gazebo>
+  </xacro:macro>
 <gazebo reference="imu_link">
     <sensor name="r2_imu" type="imu">
@@ -243,3 +113,26 @@
     </sensor>
 </gazebo>
+    <gazebo reference="camera_link">
+        <material>Gazebo/Red</material>
+        <sensor name="camera" type="camera">
+            <pose> 0 0 0 0 0 0 </pose>
+            <visualize>true</visualize>
+            <update_rate>10</update_rate>
+            <camera>
+                <horizontal_fov>1.089</horizontal_fov>
+                <image>
+                    <format>R8G8B8</format>
+                    <width>640</width>
+                    <height>480</height>
+                </image>
+                <clip>
+                    <near>0.05</near>
+                    <far>8.0</far>
+                </clip>
+            </camera>
+            <plugin name="camera_controller" filename="libgazebo_ros_camera.so">
+                <frame_name>camera_link_optical</frame_name>
+            </plugin>
+        </sensor>
+    </gazebo>
 </robot>

File: r2_description/description/r2.urdf.xacro (robot description, xacro)
@@ -5,3 +5,9 @@
     <xacro:r2/>
     <xacro:include filename="gazebo.xacro"/>
+    <xacro:luna prefix="lidar_fl_1"/>
+    <xacro:luna prefix="lidar_fr_1"/>
+    <xacro:luna prefix="lidar_lf_1"/>
+    <xacro:luna prefix="lidar_lb_1"/>
+    <xacro:luna prefix="lidar_rb_1"/>
+    <xacro:luna prefix="lidar_rf_1"/>
 </robot>

Commit message: add imu sensor on r2

File: r2_description/description/body/r2.xacro (robot description, xacro)
@@ -380,4 +380,30 @@
         </joint>
         <link name="camera_link_optical"></link>
+            <!-- IMU LINK AT CENTER OF ROBOT -->
+    <joint name="imu_joint" type="fixed">
+      <parent link="base_link" />
+      <child link="imu_link" />
+      <origin xyz="0 0 0.01" rpy="0 0 0" />
+    </joint>
+  <link name="imu_link">
+      <visual>
+          <origin xyz="0 0 0" rpy="0 0 0" />
+          <geometry>
+              <box size="0.02 0.02 0.02" />
+          </geometry>
+          <material name="grey" />
+      </visual>
+      <collision>
+          <origin xyz="0 0 0" rpy="0 0 0" />
+          <geometry>
+              <box size="0.02 0.02 0.02" />
+          </geometry>
+      </collision>
+      <inertial>
+      <origin xyz="0.0 0.0 0.0" rpy="0.0 0.0 0.0"/>
+      <mass value="0.100"/>
+      <xacro:box_inertia m="0.100" x="0.02" y="0.02" z="0.02"/>
+      </inertial>
+</link>
     </xacro:macro>
 </robot>

Commit message: change the position of camera

File: r2_description/description/body/r2.xacro (robot description, xacro)
@@ -364,5 +364,5 @@
             <parent link="base_link" />
             <child link="camera_link"/>
-            <origin xyz="0.305 0 0.08" rpy="0 0 0"/>
+            <origin xyz="0.1532118051906009 0.1 0.01867267064366568" rpy="0 0 0"/>
         </joint>
         <link name="camera_link">

Commit message: added revolute joints in r2 claw

File: r2_description/description/body/r2.xacro (robot description, xacro)
@@ -349,15 +349,17 @@
             <limit upper="0.546" lower="0.0" effort="100" velocity="100"/>
           </joint>
-          <joint name="claw_left_lift" type="continuous">
+          <joint name="claw_left_lift" type="revolute">
             <origin xyz="0.09204 -0.024511 0.0225" rpy="0 0 0"/>
             <parent link="lift_1"/>
             <child link="claw_left_1"/>
             <axis xyz="0.0 0.0 1.0"/>
-          </joint>
-          <joint name="claw_right_lift" type="continuous">
+            <limit lower="0" upper="${PI/4}" effort="4.0" velocity="0.0"/>
+          </joint>
+          <joint name="claw_right_lift" type="revolute">
             <origin xyz="0.09204 -0.060511 0.0225" rpy="0 0 -0.3"/>
             <parent link="lift_1"/>
             <child link="claw_right_1"/>
             <axis xyz="0.0 0.0 1.0"/>
+            <limit lower="0" upper="${-PI/4}" effort="4.0" velocity="0.0"/>
           </joint>
         <joint name="camera_joint" type="fixed">
@@ -371,5 +373,5 @@
                     <box size="0.010 0.03 0.03"/>
                 </geometry>
-                <material name="red"/>
+                <material name="silver"/>
             </visual>
         </link>

File: r2_description/description/common.xacro (robot description, xacro)
@@ -60,4 +60,5 @@
   </gazebo>
 <xacro:property name="M_PI" value="3.1415926535897931" />
+<xacro:property name="PI" value="3.1415926535897931" />
 <xacro:property name="M_PI_2" value="1.570796327" />
 <xacro:property name="DEG_TO_RAD" value="0.017453293" />

Commit message: added ros2 control for gripper controls
+  effort controller
+ joint position controller
- old urdf files

File: r2_description/description/body/r2.xacro (robot description, xacro)
@@ -293,4 +293,5 @@
             <child link="wheel_fl_1"/>
             <axis xyz="0.0 1.0 -0.0"/>
+            <limit upper="${2 * PI}" lower="0.0" effort="100" velocity="100"/>
           </joint>
           <joint name="wheel_bl_base" type="continuous">
@@ -299,4 +300,5 @@
             <child link="wheel_bl_1"/>
             <axis xyz="0.0 1.0 -0.0"/>
+            <limit upper="${2 * PI}" lower="0.0" effort="100" velocity="100"/>
           </joint>
           <joint name="wheel_fr_base" type="continuous">
@@ -305,4 +307,5 @@
             <child link="wheel_fr_1"/>
             <axis xyz="-0.0 -1.0 0.0"/>
+            <limit upper="${2 * PI}" lower="0.0" effort="100" velocity="100"/>
           </joint>
           <joint name="wheel_br_base" type="continuous">
@@ -311,4 +314,5 @@
             <child link="wheel_br_1"/>
             <axis xyz="-0.0 -1.0 0.0"/>
+            <limit upper="${2 * PI}" lower="0.0" effort="100" velocity="100"/>
           </joint>
           <joint name="lidar_lf" type="fixed">
@@ -354,12 +358,12 @@
             <child link="claw_left_1"/>
             <axis xyz="0.0 0.0 1.0"/>
-            <limit lower="0" upper="${PI/4}" effort="4.0" velocity="0.0"/>
+            <limit lower="0" upper="${PI/4}" effort="4.0" velocity="10.0"/>
           </joint>
           <joint name="claw_right_lift" type="revolute">
-            <origin xyz="0.09204 -0.060511 0.0225" rpy="0 0 -0.3"/>
+            <origin xyz="0.09204 -0.060511 0.0225" rpy="0 0 0"/>
             <parent link="lift_1"/>
             <child link="claw_right_1"/>
-            <axis xyz="0.0 0.0 1.0"/>
-            <limit lower="0" upper="${-PI/4}" effort="4.0" velocity="0.0"/>
+            <axis xyz="0.0 0.0 -1.0"/>
+            <limit lower="0" upper="${PI/4}" effort="4.0" velocity="10.0"/>
           </joint>
         <joint name="camera_joint" type="fixed">

File: r2_description/description/gazebo.xacro (robot description, xacro)
@@ -1,4 +1,12 @@
 <?xml version="1.0"?>
 <robot xmlns:xacro="http://www.ros.org/wiki/xacro" name="r2">
+    <gazebo>
+        <plugin filename="libgazebo_ros2_control.so" name="gz_ros2_control">
+          <robot_param>robot_description</robot_param>
+          <robot_param_node>robot_state_publisher</robot_param_node>
+          <parameters>$(find r2_description)/config/controller.yaml</parameters>
+          <controller_manager_name>r2_controller_manager</controller_manager_name>
+        </plugin>
+    </gazebo>
     <gazebo>
         <plugin name="planar_move_plugin" filename="libgazebo_ros_planar_move.so">
@@ -16,5 +24,4 @@
         <sensor name="${prefix}" type="ray">
             <always_on>true</always_on>
-            <visualize>true</visualize>
             <pose>0.0 0 0.0 0 0 0</pose>
             <update_rate>5</update_rate>
@@ -117,5 +124,4 @@
         <sensor name="camera" type="camera">
             <pose> 0 0 0 0 0 0 </pose>
-            <visualize>true</visualize>
             <update_rate>10</update_rate>
             <camera>

File: r2_description/description/r2.urdf.xacro (robot description, xacro)
@@ -11,3 +11,4 @@
     <xacro:luna prefix="lidar_rb_1"/>
     <xacro:luna prefix="lidar_rf_1"/>
+    <xacro:include filename="control.xacro"/>
 </robot>
