Commit message: fixed gazebo ball bounce issue
drastically increased gripper friction
gripper prevented from closing completely
+ simulation.launch.py launch argument to toggle worlds

File: r2_description/description/body/r2.xacro (robot description, xacro)
@@ -269,6 +269,6 @@
                 <friction>
                   <ode>
-                    <mu>0.01</mu>
-                    <mu2>0.01</mu2>
+                    <mu>10000</mu>
+                    <mu2>10000</mu2>
                   </ode>
                 </friction>
@@ -297,6 +297,6 @@
                 <friction>
                   <ode>
-                    <mu>0.01</mu>
-                    <mu2>0.01</mu2>
+                    <mu>10000</mu>
+                    <mu2>10000</mu2>
                   </ode>
                 </friction>
@@ -367,5 +367,5 @@
             <child link="lift_1"/>
             <axis xyz="0.0 0.0 1.0"/>
-            <limit upper="0.546" lower="0.0" effort="100" velocity="100"/>
+            <limit upper="0.546" lower="0.0" effort="100" velocity="1"/>
           </joint>
           <joint name="claw_left_lift" type="revolute">
@@ -374,5 +374,5 @@
             <child link="claw_left_1"/>
             <axis xyz="0.0 0.0 1.0"/>
-            <limit lower="0" upper="${PI/4}" effort="4.0" velocity="10.0"/>
+            <limit lower="0.015" upper="${PI/4}" effort="10000.0" velocity="10.0"/>
           </joint>
           <joint name="claw_right_lift" type="revolute">
@@ -381,5 +381,5 @@
             <child link="claw_right_1"/>
             <axis xyz="0.0 0.0 -1.0"/>
-            <limit lower="0" upper="${PI/4}" effort="4.0" velocity="10.0"/>
+            <limit lower="0.015" upper="${PI/4}" effort="10000.0" velocity="10.0"/>
           </joint>
         <joint name="camera_joint" type="fixed">

Commit message: increased simulation mass to prevent yaw fly issue

File: r2_description/description/body/r2.xacro (robot description, xacro)
@@ -11,5 +11,5 @@
             <inertial>
               <origin xyz="0.05532118051906009 0.005032766073950176 0.04867267064366568" rpy="0 0 0"/>
-              <mass value="23.428910512481483"/>
+              <mass value="100.428910512481483"/>
               <inertia ixx="1.172295" iyy="1.33557" izz="0.888889" ixy="-0.018699" iyz="-0.060797" ixz="-0.277735"/>
             </inertial>

Commit message: integrated silo deciding server and +capture point
+ capture point to be known to see all silos at once

File: r2_description/description/body/r2.xacro (robot description, xacro)
@@ -148,5 +148,5 @@
             </collision>
           </link>
-          <link name="lidar_fl_1">
+          <link name="luna_fl">
             <inertial>
               <origin xyz="0.005000000000005944 2.326098280241995e-07 5.689893001203927e-16" rpy="0 0 0"/>
@@ -157,5 +157,5 @@
               <origin xyz="-0.205 -0.115382 0.086" rpy="0 0 0"/>
               <geometry>
-                <mesh filename="file://$(find r2_description)/meshes/lidar_fl_1.stl" scale="0.001 0.001 0.001"/>
+                <mesh filename="file://$(find r2_description)/meshes/luna_fl.stl" scale="0.001 0.001 0.001"/>
               </geometry>
               <material name="silver"/>
@@ -164,9 +164,9 @@
               <origin xyz="-0.205 -0.115382 0.086" rpy="0 0 0"/>
               <geometry>
-                <mesh filename="file://$(find r2_description)/meshes/lidar_fl_1.stl" scale="0.001 0.001 0.001"/>
-              </geometry>
-            </collision>
-          </link>
-          <link name="lidar_fr_1">
+                <mesh filename="file://$(find r2_description)/meshes/luna_fl.stl" scale="0.001 0.001 0.001"/>
+              </geometry>
+            </collision>
+          </link>
+          <link name="luna_fr">
             <inertial>
               <origin xyz="0.005000000000008192 -3.275974437833007e-07 4.996003610813204e-16" rpy="0 0 0"/>
@@ -177,5 +177,5 @@
               <origin xyz="-0.205 0.152509 0.086" rpy="0 0 0"/>
               <geometry>
-                <mesh filename="file://$(find r2_description)/meshes/lidar_fr_1.stl" scale="0.001 0.001 0.001"/>
+                <mesh filename="file://$(find r2_description)/meshes/luna_fr.stl" scale="0.001 0.001 0.001"/>
               </geometry>
               <material name="silver"/>
@@ -184,9 +184,9 @@
               <origin xyz="-0.205 0.152509 0.086" rpy="0 0 0"/>
               <geometry>
-                <mesh filename="file://$(find r2_description)/meshes/lidar_fr_1.stl" scale="0.001 0.001 0.001"/>
-              </geometry>
-            </collision>
-          </link>
-          <link name="lidar_rf_1">
+                <mesh filename="file://$(find r2_description)/meshes/luna_fr.stl" scale="0.001 0.001 0.001"/>
+              </geometry>
+            </collision>
+          </link>
+          <link name="luna_rf">
             <inertial>
               <origin xyz="-2.0882421542661733e-07 -0.004999999999998284 1.942890293094024e-15" rpy="0 0 0"/>
@@ -197,5 +197,5 @@
               <origin xyz="-0.052465 0.19 0.0745" rpy="0 0 -${pi/2}"/>
               <geometry>
-                <mesh filename="file://$(find r2_description)/meshes/lidar_rf_1.stl" scale="0.001 0.001 0.001"/>
+                <mesh filename="file://$(find r2_description)/meshes/luna_rf.stl" scale="0.001 0.001 0.001"/>
               </geometry>
               <material name="silver"/>
@@ -204,9 +204,9 @@
               <origin xyz="-0.052465 0.19 0.0745" rpy="0 0 -${pi/2}"/>
               <geometry>
-                <mesh filename="file://$(find r2_description)/meshes/lidar_rf_1.stl" scale="0.001 0.001 0.001"/>
-              </geometry>
-            </collision>
-          </link>
-          <link name="lidar_rb_1">
+                <mesh filename="file://$(find r2_description)/meshes/luna_rf.stl" scale="0.001 0.001 0.001"/>
+              </geometry>
+            </collision>
+          </link>
+          <link name="luna_rb">
             <inertial>
               <origin xyz="-2.0882421544743401e-07 -0.004999999999999394 2.040034807748725e-15" rpy="0 0 0"/>
@@ -217,5 +217,5 @@
               <origin xyz="0.047535 0.19 0.0745" rpy="0 0 -${pi/2}"/>
               <geometry>
-                <mesh filename="file://$(find r2_description)/meshes/lidar_rb_1.stl" scale="0.001 0.001 0.001"/>
+                <mesh filename="file://$(find r2_description)/meshes/luna_rb.stl" scale="0.001 0.001 0.001"/>
               </geometry>
               <material name="silver"/>
@@ -224,5 +224,5 @@
               <origin xyz="0.047535 0.19 0.0745" rpy="0 0 -${pi/2}"/>
               <geometry>
-                <mesh filename="file://$(find r2_description)/meshes/lidar_rb_1.stl" scale="0.001 0.001 0.001"/>
+                <mesh filename="file://$(find r2_description)/meshes/luna_rb.stl" scale="0.001 0.001 0.001"/>
               </geometry>
             </collision>
@@ -345,20 +345,20 @@
             <origin xyz="0.205 0.115382 -0.086" rpy="0 0 0"/>
             <parent link="base_link"/>
-            <child link="lidar_fl_1"/>
+            <child link="luna_fl"/>
           </joint>
           <joint name="lidar_fr" type="fixed">
             <origin xyz="0.205 -0.152509 -0.086" rpy="0 0 0"/>
             <parent link="base_link"/>
-            <child link="lidar_fr_1"/>
+            <child link="luna_fr"/>
           </joint>
           <joint name="lidar_rf" type="fixed">
             <origin xyz="0.052465 -0.19 -0.0745" rpy="0 0 -${pi/2}"/>
             <parent link="base_link"/>
-            <child link="lidar_rf_1"/>
+            <child link="luna_rf"/>
           </joint>
           <joint name="lidar_rb" type="fixed">
             <origin xyz="-0.047535 -0.19 -0.0745" rpy="0 0 -${pi/2}"/>
             <parent link="base_link"/>
-            <child link="lidar_rb_1"/>
+            <child link="luna_rb"/>
           </joint>
           <joint name="lift_base_link" type="prismatic">

File: r2_description/description/common.xacro (robot description, xacro)
@@ -38,14 +38,14 @@
     <material>Gazebo/Silver</material>
   </gazebo>
-  <gazebo reference="lidar_fl_1">
+  <gazebo reference="luna_fl">
     <material>Gazebo/Silver</material>
   </gazebo>
-  <gazebo reference="lidar_fr_1">
+  <gazebo reference="luna_fr">
     <material>Gazebo/Silver</material>
   </gazebo>
-  <gazebo reference="lidar_rf_1">
+  <gazebo reference="luna_rf">
     <material>Gazebo/Silver</material>
   </gazebo>
-  <gazebo reference="lidar_rb_1">
+  <gazebo reference="luna_rb">
     <material>Gazebo/Silver</material>
   </gazebo>

File: r2_description/description/gazebo.xacro (robot description, xacro)
@@ -19,5 +19,12 @@
             <robotBaseFrame>base_footprint</robotBaseFrame>
         </plugin>
-  </gazebo>
+        <plugin name="gazebo_ros_state" filename="libgazebo_ros_state.so">
+            <ros>
+              <namespace>/demo</namespace>
+              <argument>model_states:=model_states_demo</argument>
+            </ros>
+            <update_rate>1.0</update_rate>
+        </plugin>
+    </gazebo>
   <xacro:macro name="luna" params="prefix">
     <gazebo reference="${prefix}">
@@ -55,5 +62,5 @@
             <plugin name="${prefix}" filename="libgazebo_ros_ray_sensor.so">
                 <ros>
-                    <namespace>distance</namespace>
+                    <namespace>/</namespace>
                     <remapping>~/out:=${prefix}</remapping>
                 </ros>

File: r2_description/description/r2.urdf.xacro (robot description, xacro)
@@ -5,10 +5,10 @@
     <xacro:r2/>
     <xacro:include filename="gazebo.xacro"/>
-    <xacro:luna prefix="lidar_fl_1"/>
-    <xacro:luna prefix="lidar_fr_1"/>
+    <xacro:luna prefix="luna_fl"/>
+    <xacro:luna prefix="luna_fr"/>
     <xacro:luna prefix="lidar_lf_1"/>
     <xacro:luna prefix="lidar_lb_1"/>
-    <xacro:luna prefix="lidar_rb_1"/>
-    <xacro:luna prefix="lidar_rf_1"/>
+    <xacro:luna prefix="luna_rb"/>
+    <xacro:luna prefix="luna_rf"/>
     <xacro:include filename="control.xacro"/>
 </robot>
