Commit message: Added Robocon r2 bot
+ Added meshes
+updated urdf

File: r2_description/description/common.xacro (robot description, xacro)
@@ -10,4 +10,7 @@
     <color rgba="0.0 0.0 0.8 1.0" />
 </material>
+<material name="silver">
+    <color rgba="0.700 0.700 0.700 1.000"/>
+  </material>
 <xacro:property name="M_PI" value="3.1415926535897931" />
 <xacro:property name="M_PI_2" value="1.570796327" />

File: r2_description/description/r2.urdf.xacro (robot description, xacro)
@@ -2,6 +2,6 @@
 <robot xmlns:xacro="http://www.ros.org/wiki/xacro" name="r2">
     <xacro:include filename="common.xacro"/>
-    <xacro:include filename="body/r2_body.xacro"/>
-    <xacro:r2_body/>
+    <xacro:include filename="body/r2.xacro"/>
+    <xacro:r2/>
     <xacro:include filename="gazebo.xacro"/>
 </robot>
